Commit message: work

File: ur7e_teleoperation/assets/ur5e.urdf (robot description, URDF)
Before this commit: robot ur5e, 13 links, 12 joints
Links:
- added link probe_link, mass 0.05; collision mesh filename=/home/deviant/IIIT_intern/src/ur7e_teleoperation/assets/mes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 scale=0.001 0.001 0.001; visual mesh filename=/home/deviant/IIIT_intern/src/ur7e_teleoperation/assets/mes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 scale=0.001 0.001 0.001
Joints:
- added joint probe_fixed_joint: type fixed, parent wrist_3_link, child probe_link, origin xyz=0 0 0.05 rpy=3.14159 0 0
