Commit message: usg images

File: ur7e_teleoperation/assets/kevin_ultrasound.urdf (robot description, URDF)
Before this commit: robot HumanModel, 103 links, 102 joints
Links:
- link L3: geometry collision box size=0.06 0.1 15.0; visual mesh filename=/home/deviant/IIIT_intern/src/ur7e_teleoperation/assets/mes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 scale=1. 1. 1.
